Commit message: upper leg motor socket tolerance increased, lower leg rotor coupler gap shape changed, lower leg coupler plate thickness increased

File: quad_urdf/urdf/quad.urdf (robot description, URDF)
Before this commit: robot quadruped, 13 links, 12 joints
Joints:
- joint back_left_hipX: origin xyz=0.11 -0.0 0.31 rpy=0 0 0 -> xyz=0.1083 0.0 0.0 rpy=0 0 0.0
- joint back_left_hipY: origin xyz=0.06 0.0 -0.042 rpy=0 1.57 0 -> xyz=0.077 0.0 -0.077 rpy=0 1.57 0.0
- joint back_left_knee: origin xyz=0.203 -0.038 0.05 rpy=0 3.14 0 -> xyz=0.203 -0.038 0.0 rpy=0 3.14 0
- joint back_right_hipX: origin xyz=0.0 -0.0 0.31 rpy=0 0 3.14 -> xyz=0.0 0.0 0.0 rpy=0 0 3.14
- joint back_right_hipY: origin xyz=0.1 0.0 -0.042 rpy=0 1.57 3.14 -> xyz=0.077 0.0 -0.077 rpy=0 1.57 3.14
- joint back_right_knee: origin xyz=0.203 -0.038 0.05 rpy=0 3.14 0 -> xyz=0.203 -0.038 0.0 rpy=0 3.14 0
- joint front_left_hipX: origin xyz=0.11 -0.0 -0.035 rpy=0 0 0 -> xyz=0.1083 -0.0 0.3491 rpy=0 0 0
- joint front_left_hipY: origin xyz=0.06 0.0 -0.042 rpy=0 1.57 0 -> xyz=0.077 0.0 -0.077 rpy=0 1.57 0
- joint front_left_knee: origin xyz=0.203 -0.038 0.05 rpy=0 3.14 0 -> xyz=0.203 -0.038 0.0 rpy=0 3.14 0
- joint front_right_hipX: origin xyz=0.0 -0.0 -0.035 rpy=0 0 3.14 -> xyz=0.0 -0.0 0.3491 rpy=0 0 3.14
- joint front_right_hipY: origin xyz=0.1 0.0 -0.042 rpy=0 1.57 3.14 -> xyz=0.077 0.0 -0.077 rpy=0 1.57 3.14
- joint front_right_knee: origin xyz=0.203 -0.038 0.05 rpy=0 3.14 0 -> xyz=0.203 -0.038 0.0 rpy=0 3.14 0

File: quad_urdf/urdf/quad_military.urdf (robot description, URDF)
Before this commit: robot quadruped, 13 links, 12 joints
Joints:
- joint back_left_hipX: origin xyz=0.11 -0.0 0.31 rpy=0 0 0 -> xyz=0.1083 0.0 0.0 rpy=0 0 0.0
- joint back_left_hipY: origin xyz=0.06 0.0 -0.042 rpy=0 1.57 0 -> xyz=0.077 0.0 -0.077 rpy=0 1.57 0.0
- joint back_left_knee: origin xyz=0.203 -0.038 0.05 rpy=0 3.14 0 -> xyz=0.203 -0.038 0.0 rpy=0 3.14 0
- joint back_right_hipX: origin xyz=0.0 -0.0 0.31 rpy=0 0 3.14 -> xyz=0.0 0.0 0.0 rpy=0 0 3.14
- joint back_right_hipY: origin xyz=0.1 0.0 -0.042 rpy=0 1.57 3.14 -> xyz=0.077 0.0 -0.077 rpy=0 1.57 3.14
- joint back_right_knee: origin xyz=0.203 -0.038 0.05 rpy=0 3.14 0 -> xyz=0.203 -0.038 0.0 rpy=0 3.14 0
- joint front_left_hipX: origin xyz=0.11 -0.0 -0.035 rpy=0 0 0 -> xyz=0.1083 -0.0 0.3491 rpy=0 0 0
- joint front_left_hipY: origin xyz=0.06 0.0 -0.042 rpy=0 1.57 0 -> xyz=0.077 0.0 -0.077 rpy=0 1.57 0
- joint front_left_knee: origin xyz=0.203 -0.038 0.05 rpy=0 3.14 0 -> xyz=0.203 -0.038 0.0 rpy=0 3.14 0
- joint front_right_hipX: origin xyz=0.0 -0.0 -0.035 rpy=0 0 3.14 -> xyz=0.0 -0.0 0.3491 rpy=0 0 3.14
- joint front_right_hipY: origin xyz=0.1 0.0 -0.042 rpy=0 1.57 3.14 -> xyz=0.077 0.0 -0.077 rpy=0 1.57 3.14
- joint front_right_knee: origin xyz=0.203 -0.038 0.05 rpy=0 3.14 0 -> xyz=0.203 -0.038 0.0 rpy=0 3.14 0
